File: board/apex/apex.kicad_sch (KiCad schematic)
At the start: 15 parts, among them J1 USB_C_Receptacle_USB2.0_16P, U1 AP7363-33D-13, U2 USBLC6-2P6

Commit message: added dark theme
Other:
- note added: "Mounting Holes 2.5mm"
- company: DelgadoTechnologies -> InFlynn Technologies
- moved on the sheet: H1, H2, H3, H4
